File: MSPM0-PCB.kicad_sch (KiCad schematic)
At the start: 1 part, among them U1 MSPM0G3507SPTR

Commit message: wip
Parts:
- added C1: 10u, Capacitor_SMD:C_0805_2012Metric, symbol Device:C
- added C2, C3: 470n, Capacitor_SMD:C_0603_1608Metric, symbol Device:C
- added R1: 0R, Resistor_SMD:R_0603_1608Metric, symbol Device:R
Connections:
- net at U1.39 (PA21/A1_7/VREF-): now also C3.1, R1.1
- net at U1.43 (PA23/VREF+): now also C3.2
- net +1V35: now reaches U1.48 (VCORE)
- net +1V35: now also C2.1
- net +3V3: now reaches U1.6 (VDD)
- net +3V3: now also C1.1
- net GND: now reaches U1.7 (VSS)
- net GND: now also C1.2, C2.2, R1.2

Commit message: save
Parts:
- added C4: 470n, Capacitor_SMD:C_0603_1608Metric, symbol Device:C
- added C5, C6: 15p, Capacitor_SMD:C_0603_1608Metric, symbol Device:C
- added J1: USB_C_Receptacle_USB2.0_16P, Connector_USB:USB_C_Receptacle_GCT_USB4105-xx-A_16P_TopMnt_Horizontal, symbol Connector:USB_C_Receptacle_USB2.0_16P
- added R2: 5k1, Resistor_SMD:R_0603_1608Metric, symbol Device:R
- added R3: 100k, Resistor_SMD:R_0603_1608Metric, symbol Device:R
- added X1: 8MHz, Crystal:Crystal_SMD_3225-4Pin_3.2x2.5mm, symbol Device:Crystal_GND24
Connections:
- net +3V3: now also R2.1
- net GND: now also C4.2, C5.2, C6.2, R3.1, X1.2, X1.4
- net HFXIN: now reaches U1.11 (PA5/HFXIN/FCC_IN)
- net HFXIN: now also C5.1, X1.1
- net HFXOUT: now reaches U1.12 (PA6/HFCLK_IN/HFXOUT)
- net HFXOUT: now also C6.1, X1.3
- net VREF-: now reaches C3.1, R1.1, U1.39 (PA21/A1_7/VREF-)
- net NRST: now reaches U1.4 (NRST)
- net NRST: now also C4.1, R2.2
- net VREF+: now reaches C3.2, U1.43 (PA23/VREF+)
- net ROSC: now reaches U1.8 (PA2/ROSC)
- net ROSC: now also R3.2
- new net: J1.A1 (GND), J1.A12 (GND), J1.B1 (GND), J1.B12 (GND)
- new net: J1.A4 (VBUS), J1.A9 (VBUS), J1.B4 (VBUS), J1.B9 (VBUS)
Other:
- moved on the sheet: C3, R1
