File: MSPM0-PCB.kicad_sch (KiCad schematic)
At the start: 12 parts, among them J1 USB_C_Receptacle_USB2.0_16P, U1 MSPM0G3507SPTR, X1 8MHz

Commit message: work on schematic
Parts:
- added C10, C9: 10u, Capacitor_SMD:C_0805_2012Metric, symbol Device:C
- added C11, C7, C8: 470n, Capacitor_SMD:C_0603_1608Metric, symbol Device:C
- added R4: 0R, Resistor_SMD:R_0603_1608Metric, symbol Device:R
- added R5, R6: 5k1, Resistor_SMD:R_0603_1608Metric, symbol Device:R
- added U2: USBLC6-2SC6, Package_TO_SOT_SMD:SOT-23-6, symbol Power_Protection:USBLC6-2SC6
- added U3: SPX3819M5-L-3-3, Package_TO_SOT_SMD:SOT-23-5, symbol Regulator_Linear:SPX3819M5-L-3-3
- J1: value USB_C_Receptacle_USB2.0_16P -> USB4216-03-A; Distributor Link 1 (none) -> https://www.mouser.ca/ProductDetail/GCT/USB4216-03-A?qs=Tc%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; Distributor Link 2 (none) -> https://www.digikey.ca/en/products/detail/gct/USB4216-03-A/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; LCSC (none) -> C37616412; Manufacturer (none) -> GCT; Manufacturer Part Number (none) -> USB4216-03-A
Connections:
- net +3V3: now also C10.1, U3.5 (OUT)
- net GND: now also J1.A1 (GND), J1.A12 (GND), J1.B1 (GND), J1.B12 (GND), J1.S1 (SHIELD), C10.2, C11.2, C7.2, C8.2, C9.2, U2.2 (GND), U3.2 (GND)
- net +VBUS: now reaches J1.A4 (VBUS), J1.A9 (VBUS), J1.B4 (VBUS), J1.B9 (VBUS)
- net +VBUS: now also C7.1, R4.1, U2.5 (VBUS)
- net at J1.A6 (D+): now also J1.B6 (D+), U2.3 (I/O2)
- net at J1.A7 (D-): now also J1.B7 (D-), U2.1 (I/O1)
- new net: C11.1, U3.4 (BP)
- new net +VBUSF: C8.1, C9.1, R4.2, U3.1 (IN), U3.3 (EN)
- no-connect marks 0 -> 2
Other:
- moved on the sheet: C1, C2, C3, C4, C5, C6, J1, R1, R2, R3, U1, X1

Commit message: wip
Parts:
- added J2: TC2030, Connector:Tag-Connect_TC2030-IDC-FP_2x03_P1.27mm_Vertical, symbol Connector:Conn_ARM_SWD_TagConnect_TC2030
Connections:
- net +3V3: now also J2.1 (VCC)
- net GND: now also R5.2, R6.2, J2.5 (GND)
- net NRST: now also J2.3 (~{RESET})
- net USBCC2: now reaches R5.1
- net USBCC2: now also J1.B5 (CC2)
- net at U1.34 (PA19/SWDIO): now also J2.2 (SWDIO)
- net at U1.35 (PA20/SWCLK): now also J2.4 (SWCLK)
- net USBCC1: now reaches J1.A5 (CC1)
- net USBCC1: now also R6.1
- net USBD+: now reaches J1.A6 (D+), J1.B6 (D+), U2.3 (I/O2)
- net USBD-: now reaches J1.A7 (D-), J1.B7 (D-), U2.1 (I/O1)
- no-connect marks 2 -> 3
Other:
- moved on the sheet: C11, C5, C6, C7, C8, R5, R6, U2

Commit message: wip
Parts:
- added C10, C8, C9: 470n, Capacitor_SMD:C_0603_1608Metric, symbol Device:C
- added FID1, FID2, FID3: Fiducial, Fiducial:Fiducial_1mm_Mask2mm, symbol Mechanical:Fiducial
- added MH1, MH2, MH3, MH4: M3, MountingHole:MountingHole_3.2mm_M3_Pad_Via, symbol Mechanical:MountingHole_Pad
- added R2, R3: 5k1, Resistor_SMD:R_0603_1608Metric, symbol Device:R
- added U4: LIS2DH, Package_LGA:LGA-14_2x2mm_P0.35mm_LayoutBorder3x4y, symbol Sensor_Motion:LIS2DH
- added U5: CH340E, Package_SO:MSOP-10_3x3mm_P0.5mm, symbol Interface_USB:CH340E
- renumbered C7 to C1, C5 to C11, C6 to C12, C4 to C13, C3 to C14, C8 to C2, C9 to C3, C11 to C4, C10 to C5, C1 to C6, C2 to C7, U2 to D1, R4 to R1, R3 to R4, R2 to R7, R1 to R8, U3 to U1, U1 to U3
Connections:
- net +3V3: now also C10.1, C8.1, C9.1, R2.1, R3.1, U4.4 (~{CS}), U4.7 (Vdd_IO), U4.8 (Vdd), U5.10 (V3), U5.7 (VCC)
- net GND: now also C10.2, C8.2, C9.2, MH1.1, MH2.1, MH3.1, MH4.1, U4.10 (GND), U4.11 (GND), U4.12 (GND), U4.13 (GND), U4.14 (GND), U4.3 (SDO), U4.9 (GND), U5.3 (GND)
- net USBD+: now also D1.6 (I/O1), U5.2 (UD-); no longer D1.3 (I/O2), J1.A6 (D+), J1.B6 (D+)
- net USBD-: now also D1.4 (I/O2), U5.1 (UD+); no longer D1.1 (I/O1), J1.A7 (D-), J1.B7 (D-)
- net UART0TX: now reaches U3.1 (PA0/FCC_IN)
- net UART0TX: now also U5.9 (RXD)
- net I2C1SCL: now reaches U3.14 (PB2)
- net I2C1SCL: now also R2.2, U4.1 (SCL/SPC)
- net I2C1SDA: now reaches U3.15 (PB3)
- net I2C1SDA: now also R3.2, U4.2 (SDA/SDI)
- net UART0RTS: now reaches U3.16 (PA8)
- net UART0RTS: now also U5.5 (~{CTS})
- net UART0CTS: now reaches U3.17 (PA9/RTC_OUT/CLK_OUT)
- net UART0CTS: now also U5.4 (~{RTS})
- net UART0RX: now reaches U3.2 (PA1)
- net UART0RX: now also U5.8 (TXD)
- net INT1: now reaches U3.22 (PB8)
- net INT1: now also U4.6 (INT1)
- net INT2: now reaches U3.23 (PB9)
- net INT2: now also U4.5 (INT2)
- net SWDIO: now reaches J2.2 (SWDIO), U3.34 (PA19/SWDIO)
- net SWCLK: now reaches J2.4 (SWCLK), U3.35 (PA20/SWCLK)
- new net USBCD+: D1.3 (I/O2), J1.A6 (D+), J1.B6 (D+)
- new net USBCD-: D1.1 (I/O1), J1.A7 (D-), J1.B7 (D-)
- no-connect marks 3 -> 33
Other:
- note added: "+3V3 LDO Regulator"
- note added: "Accelerometer"
- note added: "MSPM0 Microcontroller"
- note added: "SWD Header"
- note added: "USB-C Connector"
- note added: "USB-UART Converter"
- moved on the sheet: C11, C12, J2, R4, R7, X1
